File: lofi.kicad_pcb (KiCad board)
At the start: 2 copper layers, 22 x 25.4 mm, 18 parts, among them J1 NRF24l01+, J2 ISP, J3 debug, SW1 Reed, U1 TPL5111, U2 MCP1711-3.3, U3 ATtiny84V

Commit message: as sent to OSHPark
Parts:
- added REF**: castellate, lofi:castellate, F.Cu at (125.1, 69.2)
- added REF**: castellate, lofi:castellate, F.Cu at (123.8, 69.2)
- added REF**: castellate, lofi:castellate, F.Cu at (122.5, 69.2)
- added REF**: castellate, lofi:castellate, F.Cu at (121.3, 69.2)
- added REF**: castellate, lofi:castellate, F.Cu at (120.0, 69.2)
- added REF**: castellate, lofi:castellate, F.Cu at (118.7, 69.2)
- added REF**: castellate, lofi:castellate, F.Cu at (117.5, 69.2)
- added REF**: castellate, lofi:castellate, F.Cu at (116.2, 69.2)
- U1: footprint Package_TO_SOT_SMD:SOT-23-6_Handsoldering -> lofi:TPL5111
- U2: footprint Package_TO_SOT_SMD:SOT-23-5_HandSoldering -> lofi:MCP1711
- moved J2 25.8 mm to (112.1, 71.3), turned to 180 degrees
- moved C3 8.77 mm to (114.8, 76.8), turned to 90 degrees
- moved U3 7.56 mm to (120.4, 77.0), turned to 90 degrees
- moved R2 4.98 mm to (116.2, 84.1), turned to 180 degrees
- moved R3 4.94 mm to (116.2, 85.7), turned to 0 degrees
- moved U1 4.77 mm to (112.4, 85.5), turned to 90 degrees
- moved R1 4.59 mm to (116.2, 87.3), turned to 0 degrees
- moved U2 3.69 mm to (113.3, 80.7)
- moved C2 2.64 mm to (111.8, 76.5)
- moved C1 0.63 mm to (114.5, 92.1), turned to 0 degrees
- turned J3 to 180 degrees
Connections:
- net Net-(J1-Pad3) renamed /CE
- net Net-(J1-Pad4) renamed /CSN
- net Net-(J1-Pad7) renamed /MISO
- J1 pad 5: Net-(J1-Pad5) -> /SCK
- J1 pad 6: Net-(J1-Pad6) -> /MOSI
- J2 pad 3: Net-(J1-Pad5) -> /MOSI
- J2 pad 4: Net-(J1-Pad6) -> /RSTn
- J2 pad 5: Net-(J2-Pad5) -> /SCK
- U3 pad 10: Net-(U1-Pad4) -> Net-(J3-Pad1)
- U3 pad 11: Net-(U1-Pad5) -> Net-(U3-Pad11)
- U3 pad 2: Net-(U3-Pad2) -> Net-(U1-Pad5)
- U3 pad 3: Net-(J3-Pad1) -> Net-(U1-Pad4)
- U3 pad 4: Net-(J2-Pad5) -> /RSTn
- U3 pad 7: Net-(J1-Pad6) -> /MOSI
- U3 pad 9: Net-(J1-Pad5) -> /SCK
Routing:
- net GND: track 0.00 -> 58.4 mm, vias 0 -> 9
- net Net-(J3-Pad1): track 12.0 -> 34.1 mm
- net /MOSI: track 0.00 -> 21.0 mm, vias 0 -> 1
- net /MISO: track 0.00 -> 16.0 mm, vias 0 -> 1
- net /RSTn: track 0.00 -> 15.5 mm
- net /SCK: track 0.00 -> 14.7 mm, vias 0 -> 1
- net Net-(R5-Pad1): track 0.00 -> 12.1 mm
- net +3V3: track 31.8 -> 40.7 mm, vias 0 -> 3
- net Net-(U1-Pad4): track 0.00 -> 8.34 mm
- net Net-(U1-Pad5): track 0.00 -> 8.22 mm
- net /CSN: track 0.00 -> 4.16 mm
- net /CE: track 0.00 -> 4.16 mm
- net Net-(R1-Pad2): track 4.51 -> 3.20 mm
- net Net-(R1-Pad1): track 4.69 -> 3.86 mm
- net Net-(R4-Pad1): track 6.10 -> 6.67 mm
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- added copper zone on B.Cu, net GND
Other:
- board text added: "lofi ver 0.1"

Commit message: version 0.2 and 0.3
Parts:
- added C4: 0.01uF, Capacitor_SMD:C_0805_2012Metric_Pad1.15x1.40mm_HandSolder, F.Cu at (123.5, 88.7)
- added R7: 10k, Resistor_SMD:R_0805_2012Metric_Pad1.15x1.40mm_HandSolder, F.Cu at (116.1, 84.9)
- C1: footprint Diode_SMD:D_2816_7142Metric -> Capacitor_SMD:C_2816_7142Metric_Pad3.20x4.45mm_HandSolder
- C2, C3: footprint Capacitor_SMD:C_0603_1608Metric -> Capacitor_SMD:C_0805_2012Metric_Pad1.15x1.40mm_HandSolder
- D1: footprint LED_SMD:LED_0603_1608Metric -> Diode_SMD:D_0805_2012Metric_Pad1.15x1.40mm_HandSolder
- R1, R2, R3, R4, R5, R6: footprint Resistor_SMD:R_0603_1608Metric -> Resistor_SMD:R_0805_2012Metric_Pad1.15x1.40mm_HandSolder
- moved R5 7.08 mm to (123.5, 90.8), turned to 0 degrees
- moved R6 5.70 mm to (124.5, 85.6), turned to 180 degrees
- moved R2 5.14 mm to (119.7, 87.9)
- moved R3 3.97 mm to (119.7, 83.9)
- moved R1 3.80 mm to (119.7, 85.9)
- moved D1 3.37 mm to (126.9, 81.9)
- moved R4 3.33 mm to (126.9, 77.7), turned to 270 degrees
- moved J3 1.01 mm to (122.6, 93.4)
- moved SW1 0.57 mm to (130.9, 82.5)
- moved C2 0.30 mm to (111.8, 76.8)
- moved C3 0.29 mm to (114.5, 76.8)
- moved C1 0.15 mm to (114.7, 92.1)
Connections:
- J3 pad 1: Net-(J3-Pad1) -> /LED
- R5 pad 1: Net-(R5-Pad1) -> /SW
- R6 pad 1: Net-(J3-Pad1) -> Net-(D1-Pad1)
- R6 pad 2: Net-(D1-Pad1) -> /LED
- U1 pad 5: Net-(U1-Pad5) -> Net-(R7-Pad2)
- U3 pad 10: Net-(J3-Pad1) -> /LED
- U3 pad 2: Net-(U1-Pad5) -> Net-(R7-Pad1)
- U3 pad 5: Net-(R5-Pad1) -> Net-(U3-Pad5)
- U3 pad 6: Net-(U3-Pad6) -> /SW
Routing:
- net Net-(J3-Pad1): track 34.1 -> 0.00 mm
- net /LED: track 0.00 -> 20.1 mm
- net Net-(R5-Pad1): track 12.1 -> 0.00 mm
- net /SW: track 0.00 -> 11.2 mm
- net Net-(U1-Pad5): track 8.22 -> 0.00 mm
- net GND: track 58.4 -> 64.7 mm, vias 9 -> 10
- net Net-(R7-Pad1): track 0.00 -> 5.39 mm
- net Net-(R7-Pad2): track 0.00 -> 5.02 mm
- net Net-(R1-Pad1): track 3.86 -> 7.77 mm
- net Net-(R5-Pad2): track 4.63 -> 7.92 mm
- net +3V3: track 40.7 -> 38.2 mm
- net Net-(U1-Pad4): track 8.34 -> 10.7 mm
- net Net-(R4-Pad1): track 6.67 -> 8.80 mm
- net Net-(D1-Pad1): track 1.92 -> 3.79 mm
- net Net-(R1-Pad2): track 3.20 -> 4.00 mm
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Other:
- board text added: "lofi ver 0.3"
- board text removed: "lofi ver 0.1"

Commit message: latest pwb version is 0.4
Parts:
- added R8: 0R, Resistor_SMD:R_0805_2012Metric_Pad1.20x1.40mm_HandSolder, F.Cu at (112.5, 86.9)
- added R9: 0R, Resistor_SMD:R_0805_2012Metric_Pad1.20x1.40mm_HandSolder, F.Cu at (112.5, 84.9)
- R1: value 44k -> DNP
- R2: value 0 -> 20k
- R3: value 44k -> 22k
- R7: value 10k -> 0R
- moved U1 2.97 mm to (115.3, 86.2)
- moved R7 2.64 mm to (118.7, 84.5)
- moved R5 2.59 mm to (126.1, 90.4)
- moved C4 2.58 mm to (126.1, 88.3)
- moved R6 2.46 mm to (127.0, 85.1), turned to 270 degrees
- moved R2 2.24 mm to (122.0, 87.7)
- moved R3 2.23 mm to (122.0, 83.7)
- moved R1 2.23 mm to (122.0, 85.7)
- moved D1 0.78 mm to (127.0, 81.1)
- moved J2 0.52 mm to (112.2, 71.8)
- moved C2 0.52 mm to (111.9, 77.3)
- moved C3 0.52 mm to (114.6, 77.3)
- moved SW1 0.52 mm to (131.0, 83.0)
- moved U3 0.52 mm to (120.5, 77.5)
- moved REF** 0.52 mm to (123.9, 69.7)
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Connections:
- U2 pad 3: /Vb -> Net-(R8-Pad1)
Routing:
- net GND: track 64.7 -> 50.3 mm, vias 10 -> 9
- net /Vb: track 17.1 -> 21.9 mm
- net Net-(R8-Pad1): track 0.00 -> 4.73 mm
- net Net-(R7-Pad2): track 5.02 -> 8.95 mm
- net Net-(R5-Pad2): track 7.92 -> 4.87 mm
- net /LED: track 20.1 -> 23.0 mm
- net Net-(R4-Pad1): track 8.80 -> 6.68 mm
- net Net-(D1-Pad1): track 3.79 -> 1.96 mm
- net Net-(U1-Pad4): track 10.7 -> 9.13 mm
- net Net-(R7-Pad1): track 5.39 -> 4.11 mm
- net +3V3: track 38.2 -> 37.2 mm
Other:
- board size 22 x 25.4 mm -> 22 x 24.9 mm
- board text added: "lofi ver 0.4"
- board text removed: "lofi ver 0.3"
