File: lofi.sch (KiCad schematic (older format))
At the start: 18 parts, among them J1 NRF24l01+, J2 ISP, J3 debug, SW1 Reed, U1 TPL5111, U2 MCP1711-3.3, U3 ATtiny84V

Commit message: as sent to OSHPark
Parts:
- U1: footprint Package_TO_SOT_SMD:SOT-23-6_Handsoldering -> lofi:TPL5111
- U2: footprint Package_TO_SOT_SMD:SOT-23-5_HandSoldering -> lofi:MCP1711
Connections:
- net labels added: CE, CSN, MISO, MOSI, RSTn, SCK
- wire segments 76 -> 85
Changed lines of the file:
@@
 F 0 "U2" H 3050 3042 50  0000 C CNN
 F 1 "MCP1711-3.3" H 3050 2951 50  0000 C CNN
-F 2 "Package_TO_SOT_SMD:SOT-23-5_HandSoldering" H 3050 3025 50  0001 C CIN
+F 2 "lofi:MCP1711" H 3050 3025 50  0001 C CIN
 F 3 "http://www.st.com/resource/en/datasheet/ld39015.pdf" H 3050 2700 50  0001 C CNN
 	1    3050 2700
@@
 F 0 "U1" H 2900 4067 50  0000 C CNN
 F 1 "TPL5111" H 2900 3976 50  0000 C CNN
-F 2 "Package_TO_SOT_SMD:SOT-23-6_Handsoldering" H 2900 3500 50  0001 C CNN
+F 2 "lofi:TPL5111" H 2900 3500 50  0001 C CNN
 F 3 "http://www.ti.com/lit/ds/symlink/tpl5111.pdf" H 1250 3850 50  0001 C CNN
 	1    2900 3700
@@
 U 1 1 5D513364
 P 6600 4100
-F 0 "U3" H 6200 4800 50  0000 C CNN
-F 1 "ATtiny84V" H 6950 4800 50  0000 C CNN
+F 0 "U3" H 6200 4750 50  0000 C CNN
+F 1 "ATtiny84V" H 6950 4750 50  0000 C CNN
 F 2 "lofi:SOIC-14" H 6600 4100 50  0001 C CIN
 F 3 "http://ww1.microchip.com/downloads/en/DeviceDoc/doc8006.pdf" H 6600 4100 50  0001 C CNN
@@
 	7500 4750 7500 4600
 Wire Wire Line
-	7500 4600 7200 4600
-Wire Wire Line
 	7200 3700 8850 3700
 Wire Wire Line
@@
 	5900 4100 6000 4100
 Wire Wire Line
-	3300 3700 6000 3700
-Wire Wire Line
-	3300 3800 6000 3800
+	3300 3700 3950 3700
+Wire Wire Line
+	3300 3800 3850 3800
 Wire Wire Line
 	4100 2600 6600 2600
@@
 Wire Wire Line
 	5300 4100 5600 4100
-NoConn ~ 6000 4600
 NoConn ~ 6000 4700
 $Comp
@@
 P 9050 5700
 F 0 "J3" H 9130 5692 50  0000 L CNN
-F 1 "debug" H 8900 5850 50  0000 L CNN
+F 1 "debug" H 8950 5800 50  0000 L CNN
 F 2 "Resistor_SMD:R_0805_2012Metric_Pad1.15x1.40mm_HandSolder" H 9050 5700 50  0001 C CNN
 F 3 "~" H 9050 5700 50  0001 C CNN
@@
 Wire Wire Line
 	7950 4600 7500 4600
-Connection ~ 7500 4600
 $Comp
 L power:GND #PWR017
@@
 	8350 4700 8350 4100
 Wire Wire Line
-	8850 5100 8050 5100
-Wire Wire Line
-	8050 5100 8050 4300
-Wire Wire Line
 	7200 4000 8150 4000
+Connection ~ 8150 4000
+Wire Wire Line
+	8150 4000 8850 4000
+Text Label 7700 3700 0    50   ~ 0
+CE
+Text Label 7700 3800 0    50   ~ 0
+CSN
+Text Label 7700 3900 0    50   ~ 0
+SCK
+Text Label 7700 4000 0    50   ~ 0
+MOSI
+Text Label 7700 4100 0    50   ~ 0
+MISO
+Text Label 7700 4300 0    50   ~ 0
+RSTn
+Wire Wire Line
+	8150 4900 8150 4000
+Wire Wire Line
+	8150 4900 8850 4900
 Wire Wire Line
 	7200 3900 8250 3900
 Wire Wire Line
-	8850 4900 8250 4900
-Wire Wire Line
-	8250 4900 8250 3900
+	8850 5000 8050 5000
+Wire Wire Line
+	8050 5000 8050 4300
+Wire Wire Line
+	8850 5100 8250 5100
+Wire Wire Line
+	8250 5100 8250 3900
 Connection ~ 8250 3900
 Wire Wire Line
 	8250 3900 8850 3900
 Wire Wire Line
-	8850 5000 8150 5000
-Wire Wire Line
-	8150 5000 8150 4000
-Connection ~ 8150 4000
-Wire Wire Line
-	8150 4000 8850 4000
+	6000 4600 3950 4600
+Wire Wire Line
+	3950 4600 3950 3700
+Wire Wire Line
+	7250 4600 7250 5250
+Wire Wire Line
+	7250 5250 3850 5250
+Wire Wire Line
+	3850 5250 3850 3800
+Wire Wire Line
+	7250 4600 7200 4600
+Wire Wire Line
+	7500 4600 7500 3300
+Wire Wire Line
+	7500 3300 5850 3300
+Wire Wire Line
+	5850 3300 5850 3800
+Wire Wire Line
+	5850 3800 6000 3800
+Connection ~ 7500 4600
+NoConn ~ 6000 3700
 $EndSCHEMATC

Commit message: version 0.2 and 0.3
Parts:
- added C4: 0.01uF, Capacitor_SMD:C_0805_2012Metric_Pad1.15x1.40mm_HandSolder, symbol Device:C
- added R7: 10k, Resistor_SMD:R_0805_2012Metric_Pad1.15x1.40mm_HandSolder, symbol Device:R
- C1: footprint Diode_SMD:D_2816_7142Metric -> Capacitor_SMD:C_2816_7142Metric_Pad3.20x4.45mm_HandSolder
- C2, C3: footprint Capacitor_SMD:C_0603_1608Metric -> Capacitor_SMD:C_0805_2012Metric_Pad1.15x1.40mm_HandSolder
- D1: footprint LED_SMD:LED_0603_1608Metric -> Diode_SMD:D_0805_2012Metric_Pad1.15x1.40mm_HandSolder
- R1, R2, R3, R4, R5, R6: footprint Resistor_SMD:R_0603_1608Metric -> Resistor_SMD:R_0805_2012Metric_Pad1.15x1.40mm_HandSolder
Connections:
- net labels added: LED, SW
- wire segments 85 -> 73
Other:
- moved on the sheet: C3, D1, J1, J2, J3, R4, R5, R6, SW1, U3

Commit message: latest pwb version is 0.4
Parts:
- added R8, R9: 0R, Resistor_SMD:R_0805_2012Metric_Pad1.20x1.40mm_HandSolder, symbol Device:R
- R1: value 44k -> DNP
- R2: value 0 -> 20k
- R3: value 44k -> 22k
- R7: value 10k -> 0R
Connections:
- net Vb: now also R8.2; no longer U2.3 (EN)
- net at R7.2, U1.5 (DRV): now also R9.1
- new net: R8.1, R9.2, U2.3 (EN)
Other:
- note added: "DNP"
- note added: "Populate R8 or R9, NOT both.\nR8 - t84 & nrf always powered (default)\nR9 - power up t84 & nrf for one show use.\nCan't use internal SRAM."
- note added: "R2 = 20k\nR3 = 22k\n284s period"
- note added: "V2 V3\n----------------------\nsw PB2 PA7\nDRV PA2 PB0\nnc1 PB0 PA2\nnc2 PA7 PB2\nPCINT0_FLAG wdFlag swFlag\nPCINT1_FLAG swFlag wdFlag"
